File: Hardware/Mainboard/projet-chat-ese/MCU.kicad_sch (KiCad schematic)
At the start: 17 parts, among them J103 Conn_ST_STDC14, J3 UART, J5 USB_C_Receptacle_USB2.0_16P, SW1 SW_SPST, U102 STM32G431CBUx, U2 USBLC6-2SC6, Y1 Crystal_GND24

Commit message: [Update] PCB
Parts:
- removed R18, R?: 10k, Resistor_SMD:R_0402_1005Metric, symbol Device:R_Small
- removed SW?: SW_Push, MainBoard:435451019820, symbol Switch:SW_Push
- added C21: 100n, Capacitor_SMD:C_0402_1005Metric, symbol Device:C_Small
- added D5: RB081LAM-20, Diode_SMD:D_SOD-128, symbol Device:D_Schottky
- J3: footprint Connector_PinHeader_2.54mm:PinHeader_1x04_P2.54mm_Vertical -> Connector_JST:JST_EH_B4B-EH-A_1x04_P2.50mm_Vertical
- SW1: footprint (none) -> Button_Switch_SMD:SW_Push_1P1T_NO_E-Switch_TL3301NxxxxxG
Connections:
- net +3.3V: now also C8.1
- net +5V: now also D5.1 (K); no longer J5.A4 (VBUS), J5.A9 (VBUS), J5.B4 (VBUS), J5.B9 (VBUS), U2.5 (VBUS)
- net GND: now also C21.2; no longer C8.1
- net ToF_SCL: now also C8.2, R4.1, SW1.2 (B), U102.46 (PB8); no longer U102.31 (PA9)
- net ToF_SDA: now also U102.47 (PB9); no longer U102.30 (PA8)
- net ToF_~{Reset}: now also U102.2 (PC13); no longer U102.29 (PC6)
- net MOT2_Imes: now reaches U102.19 (PB2)
- net BT_UART_RX: now reaches U102.22 (PB10)
- net BT_UART_TX: now reaches U102.24 (PB11)
- net BT_~{RST}: now reaches U102.25 (PB12)
- net BT_UART_RTS: now reaches U102.26 (PB13)
- net BT_UART_CTS: now reaches U102.27 (PB14)
- net MOT2_A: now reaches U102.8 (PA0)
- net MOT2_B: now reaches U102.9 (PA1)
- net MOT_REV: no longer names the net of U102.38 (PA15)
- net Tof_SelectB renamed MOT1_Imes
- new net MOT1_A: U102.31 (PA9)
- new net MOT1_B: U102.30 (PA8)
- new net VBUS: C21.1, D5.2 (A), J5.A4 (VBUS), J5.A9 (VBUS), J5.B4 (VBUS), J5.B9 (VBUS), U2.5 (VBUS)
- no-connect marks 21 -> 13
Other:
- note added: "SCHOTTKY OR with BUCK 5V"
- note added: "USB_C"
- note removed: "Ajouter un encodeur pour une 2e roue"
- note removed: "Installer le PD"
- note removed: "PENSER A FILTER L'ENTREE PENSER A SCHOTTKY OR"
- note removed: "Rajouter un schéma de passe bas cf CDFR"
- note removed: "USB_C 3.3V"
- moved on the sheet: C8, R4, SW1
