File: Hardware/Mainboard/projet-chat-ese/projet-chat-ese.kicad_pcb (KiCad board)
At the start: 2 copper layers, 67 parts, among them J103 Conn_ST_STDC14, J2 Conn_01x06_Socket, J201 Conn_01x06_Socket, J3 UART, J5 USB_C_Receptacle_USB2.0_16P, U1 BM71BLES1FC2-0B04AA, U102 STM32G431CBUx, U2 USBLC6-2SC6, U201 ZXBM5210-SP-13, U3 ADXL343BCCZ-RL, U4 TCA9548APWR, U5 MP1475SGJ-P, U6 ZXBM5210-SP-13, U7 GO 10-SME/SP3, U8 GO 10-SME/SP3

Commit message: KSA : PCB G431 :
Parts:
- removed BU33SD5WG-TR2: LM1117DT-3.3, Package_TO_SOT_SMD:SOT-23-5
- removed C1, C2: 1u, Capacitor_SMD:C_0603_1608Metric_Pad1.08x0.95mm_HandSolder
- removed D2: GR, LED_SMD:LED_0603_1608Metric
- removed J2: Conn_01x06_Socket, Connector_JST:JST_EH_B6B-EH-A_1x06_P2.50mm_Vertical
- removed R5: 1k, Resistor_SMD:R_0402_1005Metric
- removed U6: ZXBM5210-SP-13, Package_SO:SOIC-8-1EP_3.9x4.9mm_P1.27mm_EP2.29x3mm
- removed U8: GO 10-SME/SP3, Package_SO:SOIC-8-1EP_3.9x4.9mm_P1.27mm_EP2.41x3.3mm
- added ?: , , F.Cu at (190.0, 54.3)
- added C203: 4.7n, Capacitor_SMD:C_0402_1005Metric, F.Cu at (169.5, 57.5)
- added C410: 4u7, Capacitor_SMD:C_0402_1005Metric, F.Cu at (170.8, 67.0)
- added C411: 100n, Capacitor_SMD:C_0402_1005Metric, F.Cu at (170.1, 66.3)
- added C412: 100n, Capacitor_SMD:C_0402_1005Metric, F.Cu at (178.0, 65.6)
- added C413: 100n, Capacitor_SMD:C_0402_1005Metric, F.Cu at (174.4, 69.8)
- added C414: 100n, Capacitor_SMD:C_0402_1005Metric, F.Cu at (170.9, 64.8)
- added C415: 100n, Capacitor_SMD:C_0402_1005Metric, F.Cu at (177.3, 64.9)
- added C416: 4u7, Capacitor_SMD:C_0402_1005Metric, F.Cu at (178.8, 66.4)
- added C603: 4.7n, Capacitor_SMD:C_0402_1005Metric, F.Cu at (189.6, 55.1)
- added C604: 47n, Capacitor_SMD:C_0402_1005Metric, F.Cu at (166.6, 56.0)
- added C605: 47n, Capacitor_SMD:C_0402_1005Metric, F.Cu at (188.0, 56.0)
- added D701: LED, LED_SMD:LED_0603_1608Metric, F.Cu at (182.4, 79.2)
- added F101: 2920L300, Custom:2920L300, B.Cu at (158.0, 74.5)
- added J501: Conn_01x04, Connector_JST:JST_EH_B4B-EH-A_1x04_P2.50mm_Vertical, F.Cu at (148.5, 64.0)
- added J502: Conn_01x04, Connector_JST:JST_EH_B4B-EH-A_1x04_P2.50mm_Vertical, F.Cu at (200.0, 56.5)
- added J503: Conn_01x04, Connector_JST:JST_EH_B4B-EH-A_1x04_P2.50mm_Vertical, F.Cu at (148.5, 78.0)
- added J504: Conn_01x04, Connector_JST:JST_EH_B4B-EH-A_1x04_P2.50mm_Vertical, F.Cu at (200.0, 70.2)
- added J601: Conn_01x06_Socket, Connector_JST:JST_EH_B6B-EH-A_1x06_P2.50mm_Vertical, F.Cu at (190.5, 49.0)
- added L101: 4u7, Inductor_SMD:L_APV_ANR5020, F.Cu at (192.7, 61.2)
- added R501: 4k7, Resistor_SMD:R_0402_1005Metric, F.Cu at (142.7, 70.2)
- added R502: 4k7, Resistor_SMD:R_0402_1005Metric, F.Cu at (142.7, 72.2)
- added R503: 4k7, Resistor_SMD:R_0402_1005Metric, F.Cu at (142.5, 67.5)
- added R504: 4k7, Resistor_SMD:R_0402_1005Metric, F.Cu at (145.8, 59.5)
- added R505: 4k7, Resistor_SMD:R_0402_1005Metric, F.Cu at (202.7, 61.4)
- added R506: 4k7, Resistor_SMD:R_0402_1005Metric, F.Cu at (145.7, 62.0)
- added R507: 4k7, Resistor_SMD:R_0402_1005Metric, F.Cu at (202.7, 58.7)
- added R508: 4k7, Resistor_SMD:R_0402_1005Metric, F.Cu at (152.0, 72.4)
- added R509: 4k7, Resistor_SMD:R_0402_1005Metric, B.Cu at (196.7, 75.6)
- added R510: 4k7, Resistor_SMD:R_0402_1005Metric, F.Cu at (151.9, 76.0)
- added R511: 4k7, Resistor_SMD:R_0402_1005Metric, B.Cu at (196.5, 72.2)
- added SW101: SW_SPDT, Custom:Interrupteur, F.Cu at (165.0, 82.7)
- added SW401: SW_SPST, Button_Switch_SMD:SW_Push_1P1T_NO_CK_KSC6xxJ, F.Cu at (163.3, 60.1)
- added U601: ZXBM5210-SP-13, Package_SO:SOIC-8-1EP_3.9x4.9mm_P1.27mm_EP2.29x3mm, B.Cu at (182.9, 54.0)
- added U602: GO 10-SME/SP3, Package_SO:SOIC-8-1EP_3.9x4.9mm_P1.27mm_EP2.41x3.3mm, B.Cu at (189.5, 54.8)
- added Y401: MCSJK-7U-16.00-10-30-80-B-30, Custom:SMD 3225, B.Cu at (167.0, 61.9)
- C101: renamed from C7; moved to B.Cu
- C102: renamed from C12; moved to B.Cu
- C105: renamed from C18; moved to B.Cu
- C301: renamed from C6; moved to B.Cu
- C302: renamed from C5; moved to B.Cu
- C401: renamed from C8; moved to B.Cu
- C402: renamed from C3; value ??p -> 12p; moved to B.Cu
- C403: renamed from C4; value ??p -> 10p; moved to B.Cu
- C701: renamed from C20; moved to B.Cu
- H101, H102, H103, H104: footprint MountingHole:MountingHole_2.5mm_Pad_TopBottom -> MountingHole:MountingHole_3.2mm_M3_DIN965_Pad_TopBottom
- J403: renamed from J3; footprint Connector_PinHeader_2.54mm:PinHeader_1x04_P2.54mm_Vertical -> Connector_JST:JST_EH_B4B-EH-A_1x04_P2.50mm_Vertical
- R301: renamed from R6; moved to B.Cu
- R401: renamed from R4; moved to B.Cu
- R402: renamed from R1; moved to B.Cu
- R403: renamed from R2; moved to B.Cu
- R601: renamed from R15; moved to B.Cu
- R602: renamed from R16; moved to B.Cu
- U201: moved to B.Cu
- U202: renamed from U7; moved to B.Cu
- U301: renamed from U3; moved to B.Cu
- U401: renamed from U102; moved to B.Cu
- U701: renamed from U1; moved to B.Cu
- moved H101 158.1 mm to (150.0, 50.0)
- moved H102 158.1 mm to (198.5, 50.0)
- moved H103 158.1 mm to (198.5, 85.0)
- moved H104 158.1 mm to (150.0, 85.0)
- moved C602 116.5 mm to (187.5, 52.8)
- moved C601 114.6 mm to (187.5, 54.4), turned to 180 degrees
- moved D103 109.4 mm to (193.9, 56.6), turned to 180 degrees
- moved BU33SD5WG-TR101 109.1 mm to (193.8, 66.9), turned to 180 degrees
- moved R104 106.6 mm to (187.0, 62.5), turned to 90 degrees
- moved R107 106.5 mm to (185.9, 62.3), turned to 90 degrees
- moved C101 106.0 mm to (195.0, 68.9), turned to 180 degrees
- moved R102 105.0 mm to (184.9, 68.4)
- moved R105 104.8 mm to (185.2, 64.8), turned to 90 degrees
- moved R106 104.2 mm to (183.6, 64.4)
- moved R602 104.1 mm to (177.8, 53.9)
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- renumbered BT1 to BT101, BU33SD5WG-TR1 to BU33SD5WG-TR101, C10 to C103, C13 to C104, C14 to C107, C16 to C108, C15 to C109, C11 to C111, C9 to C202, C105 to C404, C21 to C405, C17 to C601, C19 to C602, D3 to D101, D1 to D102, D6 to D103, D5 to D401, J103 to J401, J5 to J402, R9 to R101, R14 to R102, R3 to R103, R10 to R104, R11 to R105, R13 to R106, R12 to R107, R8 to R201, R201 to R202, R7 to R701, U5 to U101, U2 to U402, U4 to U501
Connections:
- C201 pad 2: +5V -> +BATT
- C202 pad 1: +5V -> +BATT
- C601 pad 2: +5V -> +BATT
- C602 pad 1: +5V -> +BATT
- R102 pad 2: GND -> Net-(U101-PG)
- R202 pad 1: +5V -> +BATT
- R602 pad 1: +5V -> +BATT
- U101 pad 1: GND -> Net-(U101-PG)
- U201 pad 2: +5V -> +BATT
- U201 pad 3: +5V -> +BATT
- U401 pad 14: /MCU/MOT1_FW -> /MCU/MOT2_FW
- U401 pad 18: /MCU/MOT1_REV -> /MCU/MOT2_REV
- U401 pad 21: +3.3VA -> +3.3V
- U401 pad 30: /MCU/MOT1_B -> /MCU/MOT2_B
- U401 pad 31: /MCU/MOT1_A -> /MCU/MOT2_A
- U401 pad 42: /MCU/USB_CC1 -> unconnected-(U401-PB4-Pad42)
- U401 pad 43: /MCU/MOT2_REV -> /MCU/MOT1_REV
- U401 pad 44: /MCU/USB_CC2 -> unconnected-(U401-PB6-Pad44)
- U401 pad 45: /MCU/MOT2_FW -> /MCU/MOT1_FW
- U401 pad 8: /MCU/MOT2_A -> /MCU/MOT1_A
- U401 pad 9: /MCU/MOT2_B -> /MCU/MOT1_B
Routing:
- net /ToF/SC0: track 0.00 -> 65.7 mm, vias 0 -> 1
- net +5V: track 0.00 -> 60.1 mm, vias 0 -> 5
- net /ToF/SC1: track 0.00 -> 55.5 mm, vias 0 -> 1
- net /ToF/SD1: track 0.00 -> 47.8 mm, vias 0 -> 1
- net +3.3V: track 0.00 -> 43.0 mm, vias 0 -> 25
- net +BATT: track 0.00 -> 42.0 mm, vias 0 -> 9
- net /MCU/MOT2_A: track 0.00 -> 26.6 mm, vias 0 -> 1
- net /MCU/MOT2_B: track 0.00 -> 24.3 mm, vias 0 -> 1
- net GND: track 0.00 -> 23.5 mm, vias 0 -> 16
- net /MCU/MOT1_Imes: track 0.00 -> 23.3 mm, vias 0 -> 3
- net /BT_Module/BT_UART_RX: track 0.00 -> 21.0 mm, vias 0 -> 2
- net /ToF/SD0: track 0.00 -> 20.8 mm
- net /MCU/MOT1_A: track 0.00 -> 20.5 mm, vias 0 -> 1
- net /MCU/MOT1_B: track 0.00 -> 20.5 mm, vias 0 -> 1
- net /ToF/SD2: track 0.00 -> 19.0 mm
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- added copper zone on B.Cu, net (none)
- added copper zone on F.Cu, net (none)
- added copper zone on In1.Cu, net (none)
- added copper zone on In2.Cu, net (none)
- added copper zone on In2.Cu, net +3.3V
- added copper zone on F.Cu, net +BATT
- added copper zone on In2.Cu, net +BATT
- added copper zone on B.Cu, net /Motor Sheet/MOT+_OUT
- added copper zone on B.Cu, net /Motor Sheet1/MOT+_OUT
- added copper zone on B.Cu, net GND
- added copper zone on F.Cu, net GND
- added copper zone on In1.Cu, net GND
- added copper zone on B.Cu, net Net-(BT101-+)
- added copper zone on B.Cu, net Net-(D101-K)
- added copper zone on F.Cu, net Net-(D103-A)
- added copper zone on F.Cu, net Net-(U101-SW)
- added copper zone on In2.Cu, net Net-(U101-SW)
Other:
- board outline added: 58.5 x 45 mm
- copper layers 2 -> 4

Commit message: On a pas de wiork trtee anyway
Parts:
- removed ?: , 
- removed C604: 47n, Capacitor_SMD:C_0402_1005Metric
- removed SW101: SW_SPDT, Custom:Interrupteur
- added C204: 100n, Capacitor_SMD:C_0402_1005Metric, F.Cu at (178.0, 60.8)
- added R203: 10m, Resistor_SMD:R_0805_2012Metric, B.Cu at (169.2, 50.1)
- added R204: 10m, Resistor_SMD:R_0805_2012Metric, B.Cu at (182.0, 52.5)
- BT101: footprint Connector_AMASS:AMASS_XT30U-F_1x02_P5.0mm_Vertical -> Connector_JST:JST_XH_B2B-XH-AM_1x02_P2.50mm_Vertical
- C105: moved to F.Cu
- C201, C202, C601, C602, D101, R201, R202, R504, R505, R506, R507: moved to B.Cu
- C203: value 4.7n -> 100n
- J201, J601: footprint Connector_JST:JST_EH_B6B-EH-A_1x06_P2.50mm_Vertical -> Connector_JST:JST_PH_B6B-PH-K_1x06_P2.00mm_Vertical
- J403, J501, J502, J503, J504: footprint Connector_JST:JST_EH_B4B-EH-A_1x04_P2.50mm_Vertical -> Connector_JST:JST_PH_B4B-PH-K_1x04_P2.00mm_Vertical
- U202, U602: value GO 10-SME/SP3 -> NCS199A3RSQT2G; footprint Package_SO:SOIC-8-1EP_3.9x4.9mm_P1.27mm_EP2.41x3.3mm -> Custom:SC70-6; moved to F.Cu
- U501: footprint Package_SO:TSSOP-24_4.4x7.8mm_P0.65mm -> Package_DFN_QFN:VQFN-24-1EP_4x4mm_P0.5mm_EP2.45x2.45mm
- moved BT101 49.8 mm to (189.8, 48.5), turned to 0 degrees
- moved F101 38.8 mm to (191.6, 55.0), turned to -90 degrees
- moved D101 37.7 mm to (194.2, 63.0), turned to -90 degrees
- moved BU33SD5WG-TR101 32.8 mm to (161.1, 68.3), turned to 90 degrees
- moved C105 30.2 mm to (161.0, 65.3), turned to 0 degrees
- moved R503 24.1 mm to (166.6, 67.5), turned to 180 degrees
- moved R502 22.8 mm to (165.0, 77.2)
- moved R501 22.0 mm to (164.5, 67.5)
- moved D103 19.1 mm to (182.4, 71.9), turned to 0 degrees
- moved C603 18.5 mm to (186.7, 73.4), turned to -90 degrees
- moved C605 16.5 mm to (188.3, 72.5), turned to 180 degrees
- moved J401 15.1 mm to (161.3, 85.3)
- moved C103 14.1 mm to (188.5, 57.2), turned to 180 degrees
- moved U602 12.1 mm to (178.0, 58.6), turned to 0 degrees
- moved C109 12.1 mm to (190.3, 69.9), turned to -90 degrees
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Connections:
- C203 pad 1: /MCU/MOT1_Imes -> GND
- C203 pad 2: GND -> +3.3V
- D101 pad 1: Net-(D101-K) -> +BATT
- F101 pad 2: Net-(D101-K) -> +BATT
- U202 pad 1: /Motor Sheet/MOT+ -> GND
- U202 pad 2: /Motor Sheet/MOT+ -> GND
- U202 pad 3: /Motor Sheet/MOT+_OUT -> +3.3V
- U202 pad 5: GND -> /Motor Sheet/MOT+
- U202 pad 6: unconnected-(U202-UREF-Pad6) -> /MCU/MOT1_Imes
- U602 pad 1: /Motor Sheet1/MOT+ -> GND
- U602 pad 2: /Motor Sheet1/MOT+ -> GND
- U602 pad 3: /Motor Sheet1/MOT+_OUT -> +3.3V
- U602 pad 5: GND -> /Motor Sheet1/MOT+
- U602 pad 6: unconnected-(U602-UREF-Pad6) -> /MCU/MOT2_Imes
Routing:
- net /ToF/SC0: track 65.7 -> 2.16 mm, vias 1 -> 0
- net +5V: track 60.1 -> 0.00 mm, vias 5 -> 0
- net /ToF/SC1: track 55.5 -> 2.42 mm, vias 1 -> 0
- net /ToF/SD1: track 47.8 -> 2.32 mm, vias 1 -> 0
- net +BATT: track 42.0 -> 1.59 mm, vias 9 -> 11
- net +3.3V: track 43.0 -> 9.95 mm, vias 25 -> 10
- net /MCU/MOT2_A: track 26.6 -> 0.00 mm, vias 1 -> 0
- net /MCU/MOT2_B: track 24.3 -> 0.00 mm, vias 1 -> 0
- net /MCU/MOT1_Imes: track 23.3 -> 0.00 mm, vias 3 -> 0
- net /BT_Module/BT_UART_RX: track 21.0 -> 0.00 mm, vias 2 -> 0
- net GND: track 23.5 -> 2.97 mm, vias 16 -> 4
- net /ToF/SD0: track 20.8 -> 2.04 mm
- net /BT_Module/BT_UART_TX: track 18.5 -> 0.00 mm, vias 2 -> 0
- net /MCU/MOT2_Imes: track 18.4 -> 0.00 mm, vias 1 -> 0
- net /MCU/USB_DP: track 17.7 -> 0.00 mm, vias 1 -> 0
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- added copper zone on B.Cu, net +BATT
- added copper zone on B.Cu, net /Motor Sheet1/MOT+
- added copper zone on F.Cu, net Net-(C108-Pad1)
- removed copper zone on B.Cu, net (none)
- removed copper zone on F.Cu, net (none)
- removed copper zone on In1.Cu, net (none)
- removed copper zone on In2.Cu, net (none)
- removed copper zone on B.Cu, net Net-(D101-K)

Commit message: Finishing PCB
Parts:
- removed C603: 4.7n, Capacitor_SMD:C_0402_1005Metric
- removed C605: 47n, Capacitor_SMD:C_0402_1005Metric
- C101, C102, C401: moved to F.Cu
- C405, R501, R503, R508, R510: moved to B.Cu
- moved D102 46.8 mm to (199.8, 80.7), turned to 180 degrees
- moved R103 45.1 mm to (199.6, 79.4), turned to 180 degrees
- moved C101 31.3 mm to (163.7, 69.1), turned to 90 degrees
- moved J403 13.6 mm to (156.4, 70.1)
- moved D401 10.2 mm to (184.2, 75.5), turned to 0 degrees
- moved R701 9.60 mm to (182.4, 86.1), turned to 90 degrees
- moved U402 4.77 mm to (184.5, 78.9), turned to 0 degrees
- moved C403 4.44 mm to (165.8, 59.6), turned to 45 degrees
- moved R503 4.32 mm to (169.5, 70.7)
- moved C405 3.96 mm to (188.6, 79.1), turned to 0 degrees
- moved D701 3.80 mm to (182.4, 83.0), turned to -90 degrees
- moved R501 3.74 mm to (167.6, 69.6)
- moved R502 3.10 mm to (165.1, 74.1)
- moved C401 2.72 mm to (157.6, 59.9)
- moved J401 2.34 mm to (163.6, 84.8)
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Connections:
- J403 pad 1: +3.3V -> +5V
- J403 pad 2: /MCU/UART1_Tx -> /MCU/UART1_Rx
- J403 pad 3: /MCU/UART1_Rx -> GND
- U201 pad 9: (no net) -> GND
- U401 pad 10: /MCU/UART1_Tx -> unconnected-(U401-PA2-Pad10)
- U401 pad 11: /MCU/UART1_Rx -> /MCU/MOT1_Imes
- U401 pad 25: /BT_Module/BT_~{RESET} -> unconnected-(U401-PB12-Pad25)
- U401 pad 28: /MCU/MOT1_Imes -> unconnected-(U401-PB15-Pad28)
- U401 pad 38: unconnected-(U401-PA15-Pad38) -> /MCU/UART1_Rx
- U401 pad 39: unconnected-(U401-PC10-Pad39) -> /BT_Module/BT_~{RESET}
- U601 pad 9: (no net) -> GND
Routing:
- net /ToF/SC0: track 2.16 -> 55.4 mm, vias 0 -> 1
- net /ToF/SD0: track 2.04 -> 52.6 mm, vias 0 -> 1
- net /ToF/SC1: track 2.42 -> 44.7 mm, vias 0 -> 1
- net +3.3V: track 9.95 -> 45.3 mm, vias 10 -> 28
- net /ToF/SD2: track 2.15 -> 37.2 mm, vias 0 -> 1
- net /MCU/NRST: track 0.00 -> 34.3 mm, vias 0 -> 1
- net /ToF/SC2: track 2.18 -> 36.4 mm, vias 0 -> 1
- net /ToF/SD1: track 2.32 -> 36.3 mm, vias 0 -> 1
- net /MCU/MOT1_REV: track 0.00 -> 31.0 mm
- net /MCU/SWO: track 0.00 -> 28.4 mm, vias 0 -> 1
- net /MCU/ToF_SCL: track 2.18 -> 30.5 mm, vias 0 -> 3
- net /MCU/MOT1_FW: track 0.00 -> 28.2 mm
- net /ToF/SD3: track 0.00 -> 26.9 mm, vias 0 -> 1
- net GND: track 2.97 -> 29.5 mm, vias 4 -> 160
- net /MCU/MOT2_B: track 0.00 -> 26.4 mm, vias 0 -> 2
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- added copper zone on F.Cu, net +5V
- added copper zone on In2.Cu, net +5V
- added copper zone on F.Cu, net VBUS
- added copper zone on In2.Cu, net VBUS

Commit message: PCB G431 details
Routing:
- net GND: vias 160 -> 166
Changed lines of the file:
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@@
 	)
 	(via
+		(at 185.4 63.8)
+		(size 0.4)
+		(drill 0.3)
+		(layers "F.Cu" "B.Cu")
+		(free yes)
+		(net 1)
+	)
+	(via
 		(at 201 87.7)
 		(size 0.4)
@@
 	)
 	(via
+		(at 192.9 77.6)
+		(size 0.4)
+		(drill 0.3)
+		(layers "F.Cu" "B.Cu")
+		(free yes)
+		(net 1)
+	)
+	(via
 		(at 173.5 78.45)
 		(size 0.4)
@@
 	)
 	(via
+		(at 169.6 56.6)
+		(size 0.4)
+		(drill 0.3)
+		(layers "F.Cu" "B.Cu")
+		(free yes)
+		(net 1)
+	)
+	(via
 		(at 173.4 46.45)
 		(size 0.4)
@@
 	)
 	(via
+		(at 181.4 57.1)
+		(size 0.4)
+		(drill 0.3)
+		(layers "F.Cu" "B.Cu")
+		(free yes)
+		(net 1)
+	)
+	(via
 		(at 158.4 88.6)
 		(size 0.4)
@@
 	)
 	(via
+		(at 174.4 77.3)
+		(size 0.4)
+		(drill 0.3)
+		(layers "F.Cu" "B.Cu")
+		(free yes)
+		(net 1)
+	)
+	(via
 		(at 202.15 71.4)
 		(size 0.4)
@@
 	)
 	(via
+		(at 164.6 65.7)
+		(size 0.4)
+		(drill 0.3)
+		(layers "F.Cu" "B.Cu")
+		(free yes)
+		(net 1)
+	)
+	(via
 		(at 157.3 56.1)
 		(size 0.4)
@@
 	)
 	(segment
-		(start 173.5 76.876674)
-		(end 173.5 72.3829)
+		(start 176.85 79.7)
+		(end 175.9 79.7)
 		(width 0.2)
 		(layer "F.Cu")
@@
 	)
 	(segment
-		(start 172.15 71.0329)
-		(end 172.15 70.6)
+		(start 177.15 80)
+		(end 176.85 79.7)
 		(width 0.2)
 		(layer "F.Cu")
@@
 	)
 	(segment
-		(start 177.2 80)
-		(end 177.15 80)
+		(start 172.15 71.0329)
+		(end 172.15 70.6)
 		(width 0.2)
 		(layer "F.Cu")
@@
 	)
 	(segment
-		(start 176.079026 79.4557)
-		(end 173.5 76.876674)
+		(start 173.5 77.3)
+		(end 173.5 72.3829)
 		(width 0.2)
 		(layer "F.Cu")
@@
 	)
 	(segment
-		(start 176.6057 79.4557)
-		(end 176.079026 79.4557)
+		(start 177.2 80)
+		(end 177.15 80)
 		(width 0.2)
 		(layer "F.Cu")
@@
 	)
 	(segment
-		(start 177.15 80)
-		(end 176.6057 79.4557)
+		(start 175.9 79.7)
+		(end 173.5 77.3)
 		(width 0.2)
 		(layer "F.Cu")
