File: Hardware/Mainboard/projet-chat-ese/accelerometer.kicad_sch (KiCad schematic)
At the start: 4 parts, among them U3 ADXL343BCCZ-RL

Commit message: [Update] PCB
Parts:
- U3: footprint LGA_CC-14-1_ADI -> Custom:LGA_CC-14-1_ADI
Changed lines of the file:
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@@
-	)
-	(junction
-		(at 102.87 95.25)
-		(diameter 0)
-		(color 0 0 0 0)
 	)
 	(junction
@@
 		(color 0 0 0 0)
 	)
-	(junction
-		(at 102.87 93.98)
-		(diameter 0)
-		(color 0 0 0 0)
-	)
-	(junction
-		(at 97.79 93.98)
-		(diameter 0)
-		(color 0 0 0 0)
+	(no_connect
+		(at 177.8 95.25)
 	)
 	(no_connect
 		(at 106.68 92.71)
 	)
-	(no_connect
-		(at 177.8 95.25)
-	)
-	(wire
-		(pts
-			(xy 102.87 93.98) (xy 102.87 95.25)
-		)
-		(stroke
-			(width 0)
-			(type default)
-		)
-	)
 	(wire
 		(pts
@@
 	(wire
 		(pts
-			(xy 96.52 93.98) (xy 97.79 93.98)
-		)
-		(stroke
-			(width 0)
-			(type default)
-		)
-	)
-	(wire
-		(pts
-			(xy 102.87 90.17) (xy 102.87 93.98)
-		)
-		(stroke
-			(width 0)
-			(type default)
-		)
-	)
-	(wire
-		(pts
 			(xy 91.44 100.33) (xy 95.25 100.33)
 		)
@@
 	(wire
 		(pts
-			(xy 97.79 93.98) (xy 102.87 93.98)
-		)
-		(stroke
-			(width 0)
-			(type default)
-		)
-	)
-	(wire
-		(pts
-			(xy 102.87 95.25) (xy 102.87 97.79)
-		)
-		(stroke
-			(width 0)
-			(type default)
-		)
-	)
-	(wire
-		(pts
 			(xy 185.42 87.63) (xy 177.8 87.63)
 		)
@@
 	(wire
 		(pts
-			(xy 102.87 97.79) (xy 106.68 97.79)
-		)
-		(stroke
-			(width 0)
-			(type default)
-		)
-	)
-	(wire
-		(pts
-			(xy 102.87 95.25) (xy 106.68 95.25)
-		)
-		(stroke
-			(width 0)
-			(type default)
-		)
-	)
-	(wire
-		(pts
 			(xy 91.44 87.63) (xy 97.79 87.63)
 		)
@@
 	(wire
 		(pts
-			(xy 106.68 90.17) (xy 102.87 90.17)
-		)
-		(stroke
-			(width 0)
-			(type default)
-		)
-	)
-	(wire
-		(pts
-			(xy 97.79 92.71) (xy 97.79 93.98)
+			(xy 142.24 115.57) (xy 142.24 118.11)
 		)
 		(stroke
@@
 	(symbol
 		(lib_id "power:GND")
-		(at 96.52 93.98 270)
+		(at 142.24 118.11 0)
+		(unit 1)
+		(exclude_from_sim no)
+		(in_bom yes)
+		(on_board yes)
+		(dnp no)
+		(fields_autoplaced yes)
+		(property "Reference" "#PWR0301"
+			(at 142.24 124.46 0)
+			(effects
+				(font
+					(size 1.27 1.27)
+				)
+				(hide yes)
+			)
+		)
+		(property "Value" "GND"
+			(at 142.24 123.19 0)
+			(effects
+				(font
+					(size 1.27 1.27)
+				)
+			)
+		)
+		(property "Footprint" ""
+			(at 142.24 118.11 0)
+			(effects
+				(font
+					(size 1.27 1.27)
+				)
+				(hide yes)
+			)
+		)
+		(property "Datasheet" ""
+			(at 142.24 118.11 0)
+			(effects
+				(font
+					(size 1.27 1.27)
+				)
+				(hide yes)
+			)
+		)
+		(property "Description" "Power symbol creates a global label with name \"GND\" , ground"
+			(at 142.24 118.11 0)
+			(effects
+				(font
+					(size 1.27 1.27)
+				)
+				(hide yes)
+			)
+		)
+		(pin "1"
+		)
+		(instances
+			(project "projet-chat-ese"
+				(path "/3d65b2f4-4354-4e18-9b77-809d2b1122a1/64873241-b38d-455e-8523-56dba9a4e972"
+					(reference "#PWR0301")
+					(unit 1)
+				)
+			)
+		)
+	)
+	(symbol
+		(lib_id "power:GND")
+		(at 97.79 92.71 0)
 		(unit 1)
 		(exclude_from_sim no)
@@
 		(fields_autoplaced yes)
 		(property "Reference" "#PWR017"
-			(at 90.17 93.98 0)
+			(at 97.79 99.06 0)
 			(effects
 				(font
@@
 		)
 		(property "Value" "GND"
-			(at 92.71 93.9799 90)
-			(effects
-				(font
-					(size 1.27 1.27)
-				)
-				(justify right)
+			(at 97.79 97.79 0)
+			(effects
+				(font
+					(size 1.27 1.27)
+				)
 			)
 		)
 		(property "Footprint" ""
-			(at 96.52 93.98 0)
+			(at 97.79 92.71 0)
 			(effects
 				(font
@@
 		)
 		(property "Datasheet" ""
-			(at 96.52 93.98 0)
+			(at 97.79 92.71 0)
 			(effects
 				(font
@@
 		)
 		(property "Description" "Power symbol creates a global label with name \"GND\" , ground"
-			(at 96.52 93.98 0)
+			(at 97.79 92.71 0)
 			(effects
 				(font
@@
 			)
 		)
-		(property "Footprint" "LGA_CC-14-1_ADI"
+		(property "Footprint" "Custom:LGA_CC-14-1_ADI"
 			(at 106.68 87.63 0)
 			(effects

Commit message: KSA : PCB G431 :
Parts:
- renumbered C6 to C301, C5 to C302, R6 to R301, U3 to U301
Changed lines of the file:
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@@
 		(dnp no)
 		(fields_autoplaced yes)
-		(property "Reference" "#PWR0301"
+		(property "Reference" "#PWR0305"
 			(at 142.24 124.46 0)
 			(effects
@@
 			(project "projet-chat-ese"
 				(path "/3d65b2f4-4354-4e18-9b77-809d2b1122a1/64873241-b38d-455e-8523-56dba9a4e972"
-					(reference "#PWR0301")
+					(reference "#PWR0305")
 					(unit 1)
 				)
@@
 		(dnp no)
 		(fields_autoplaced yes)
-		(property "Reference" "#PWR017"
+		(property "Reference" "#PWR0304"
 			(at 97.79 99.06 0)
 			(effects
@@
 			(project "projet-chat-ese"
 				(path "/3d65b2f4-4354-4e18-9b77-809d2b1122a1/64873241-b38d-455e-8523-56dba9a4e972"
-					(reference "#PWR017")
+					(reference "#PWR0304")
 					(unit 1)
 				)
@@
 		(dnp no)
 		(fields_autoplaced yes)
-		(property "Reference" "#PWR018"
+		(property "Reference" "#PWR0303"
 			(at 95.25 114.3 0)
 			(effects
@@
 			(project "projet-chat-ese"
 				(path "/3d65b2f4-4354-4e18-9b77-809d2b1122a1/64873241-b38d-455e-8523-56dba9a4e972"
-					(reference "#PWR018")
+					(reference "#PWR0303")
 					(unit 1)
 				)
@@
 		(dnp no)
 		(fields_autoplaced yes)
-		(property "Reference" "#PWR016"
+		(property "Reference" "#PWR0302"
 			(at 95.25 100.33 0)
 			(effects
@@
 			(project "projet-chat-ese"
 				(path "/3d65b2f4-4354-4e18-9b77-809d2b1122a1/64873241-b38d-455e-8523-56dba9a4e972"
-					(reference "#PWR016")
+					(reference "#PWR0302")
 					(unit 1)
 				)
@@
 		(on_board yes)
 		(dnp no)
-		(property "Reference" "C6"
+		(property "Reference" "C301"
 			(at 92.71 104.1462 0)
 			(effects
@@
 			(project "projet-chat-ese"
 				(path "/3d65b2f4-4354-4e18-9b77-809d2b1122a1/64873241-b38d-455e-8523-56dba9a4e972"
-					(reference "C6")
+					(reference "C301")
 					(unit 1)
 				)
@@
 		(dnp no)
 		(fields_autoplaced yes)
-		(property "Reference" "U3"
+		(property "Reference" "U301"
 			(at 142.24 77.47 0)
 			(effects
@@
 			(project "projet-chat-ese"
 				(path "/3d65b2f4-4354-4e18-9b77-809d2b1122a1/64873241-b38d-455e-8523-56dba9a4e972"
-					(reference "U3")
+					(reference "U301")
 					(unit 1)
 				)
@@
 		(on_board yes)
 		(dnp no)
-		(property "Reference" "C5"
+		(property "Reference" "C302"
 			(at 95.25 88.9062 0)
 			(effects
@@
 			(project ""
 				(path "/3d65b2f4-4354-4e18-9b77-809d2b1122a1/64873241-b38d-455e-8523-56dba9a4e972"
-					(reference "C5")
+					(reference "C302")
 					(unit 1)
 				)
@@
 		(dnp no)
 		(fields_autoplaced yes)
-		(property "Reference" "#PWR014"
+		(property "Reference" "#PWR0306"
 			(at 195.58 92.71 0)
 			(effects
@@
 			(project ""
 				(path "/3d65b2f4-4354-4e18-9b77-809d2b1122a1/64873241-b38d-455e-8523-56dba9a4e972"
-					(reference "#PWR014")
+					(reference "#PWR0306")
 					(unit 1)
 				)
@@
 		(on_board yes)
 		(dnp no)
-		(property "Reference" "R6"
+		(property "Reference" "R301"
 			(at 182.88 97.79 90)
 			(effects
@@
 			(project ""
 				(path "/3d65b2f4-4354-4e18-9b77-809d2b1122a1/64873241-b38d-455e-8523-56dba9a4e972"
-					(reference "R6")
+					(reference "R301")
 					(unit 1)
 				)
@@
 		(dnp no)
 		(fields_autoplaced yes)
-		(property "Reference" "#PWR015"
+		(property "Reference" "#PWR0301"
 			(at 95.25 87.63 0)
 			(effects
@@
 			(project ""
 				(path "/3d65b2f4-4354-4e18-9b77-809d2b1122a1/64873241-b38d-455e-8523-56dba9a4e972"
-					(reference "#PWR015")
-					(unit 1)
-				)
+					(reference "#PWR0301")
+					(unit 1)
+				)

Commit message: check pcb kenny LF
Other:
- moved on the sheet: C301, C302
Changed lines of the file:
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@@
+	(wire
+		(pts
+			(xy 185.42 102.87) (xy 177.8 102.87)
+		)
+		(stroke
+			(width 0)
+			(type default)
+		)
+	)
+	(wire
+		(pts
+			(xy 185.42 90.17) (xy 177.8 90.17)
+		)
+		(stroke
+			(width 0)
+			(type default)
+		)
+	)
+	(wire
+		(pts
+			(xy 185.42 87.63) (xy 177.8 87.63)
+		)
+		(stroke
+			(width 0)
+			(type default)
+		)
+	)
+	(wire
+		(pts
+			(xy 177.8 92.71) (xy 180.34 92.71)
+		)
+		(stroke
+			(width 0)
+			(type default)
+		)
+	)
+	(wire
+		(pts
+			(xy 185.42 100.33) (xy 177.8 100.33)
+		)
+		(stroke
+			(width 0)
+			(type default)
+		)
+	)
 	(wire
 		(pts
 			(xy 97.79 87.63) (xy 106.68 87.63)
-		)
-		(stroke
-			(width 0)
-			(type default)
-		)
-	)
-	(wire
-		(pts
-			(xy 185.42 102.87) (xy 177.8 102.87)
-		)
-		(stroke
-			(width 0)
-			(type default)
-		)
-	)
-	(wire
-		(pts
-			(xy 185.42 90.17) (xy 177.8 90.17)
-		)
-		(stroke
-			(width 0)
-			(type default)
-		)
-	)
-	(wire
-		(pts
-			(xy 185.42 87.63) (xy 177.8 87.63)
-		)
-		(stroke
-			(width 0)
-			(type default)
-		)
-	)
-	(wire
-		(pts
-			(xy 177.8 92.71) (xy 180.34 92.71)
-		)
-		(stroke
-			(width 0)
-			(type default)
-		)
-	)
-	(wire
-		(pts
-			(xy 185.42 100.33) (xy 177.8 100.33)
 		)
 		(stroke
@@
 	(symbol
 		(lib_id "Device:C_Small")
-		(at 95.25 105.41 0)
+		(at 97.79 90.17 0)
 		(mirror y)
 		(unit 1)
@@
 		(dnp no)
 		(property "Reference" "C301"
-			(at 92.71 104.1462 0)
+			(at 95.25 88.9062 0)
 			(effects
 				(font
@@
 		)
 		(property "Value" "100n"
-			(at 92.71 106.6862 0)
+			(at 95.25 91.4462 0)
 			(effects
 				(font
@@
 		)
 		(property "Footprint" "Capacitor_SMD:C_0402_1005Metric"
-			(at 95.25 105.41 0)
+			(at 97.79 90.17 0)
 			(effects
 				(font
@@
 		)
 		(property "Datasheet" "~"
-			(at 95.25 105.41 0)
+			(at 97.79 90.17 0)
 			(effects
 				(font
@@
 		)
 		(property "Description" "Unpolarized capacitor, small symbol"
-			(at 95.25 105.41 0)
+			(at 97.79 90.17 0)
 			(effects
 				(font
@@
 	(symbol
 		(lib_id "Device:C_Small")
-		(at 97.79 90.17 0)
+		(at 95.25 105.41 0)
 		(mirror y)
 		(unit 1)
@@
 		(dnp no)
 		(property "Reference" "C302"
-			(at 95.25 88.9062 0)
+			(at 92.71 104.1462 0)
 			(effects
 				(font
@@
 		)
 		(property "Value" "1u"
-			(at 95.25 91.4462 0)
+			(at 92.71 106.6862 0)
 			(effects
 				(font
@@
 		)
 		(property "Footprint" "Capacitor_SMD:C_0603_1608Metric"
-			(at 97.79 90.17 0)
+			(at 95.25 105.41 0)
 			(effects
 				(font
@@
 		)
 		(property "Datasheet" "~"
-			(at 97.79 90.17 0)
+			(at 95.25 105.41 0)
 			(effects
 				(font
@@
 		)
 		(property "Description" "Unpolarized capacitor, small symbol"
-			(at 97.79 90.17 0)
-			(effects
-				(font
+			(at 95.25 105.41 0)
+			(effects
+				(font
