File: Hardware/Mainboard/projet-chat-ese/projet-chat-ese.kicad_sch (KiCad schematic)
At the start: 4 parts

Commit message: [Update] PCB
Parts:
- added BT1: Battery, Connector_AMASS:AMASS_XT30U-F_1x02_P5.0mm_Vertical, symbol Device:Battery
- added BU33SD5WG-TR1, BU33SD5WG-TR2: LM1117DT-3.3, Package_TO_SOT_SMD:SOT-23-5, symbol Regulator_Linear:MCP1802x-xx02xOT
- added C1, C18, C2, C7: 1u, Capacitor_SMD:C_0603_1608Metric_Pad1.08x0.95mm_HandSolder, symbol Device:C_Small
- added C10, C11, C15: 22u, Capacitor_SMD:C_0805_2012Metric, symbol Device:C_Small
- added C12, C13, C14: 100n, Capacitor_SMD:C_0402_1005Metric, symbol Device:C_Small
- added C16: 15p, Capacitor_SMD:C_0402_1005Metric, symbol Device:C_Small
- added D1, D2: GR, LED_SMD:LED_0603_1608Metric, symbol Device:LED
- added D3, D6: RB081LAM-20, Diode_SMD:D_SOD-128, symbol Device:D_Schottky
- added F1: 2920L300, symbol Device:Fuse
- added L1: 4u7, symbol Device:L_Small
- added R10: 20, Resistor_SMD:R_0402_1005Metric, symbol Device:R_Small
- added R11: 16k, Resistor_SMD:R_0402_1005Metric, symbol Device:R_Small
- added R12: 40.2k, Resistor_SMD:R_0402_1005Metric, symbol Device:R_Small
- added R13: 7.68k, Resistor_SMD:R_0402_1005Metric, symbol Device:R_Small
- added R14, R9: 100k, Resistor_SMD:R_0402_1005Metric, symbol Device:R_Small
- added R3, R5: 1k, Resistor_SMD:R_0402_1005Metric, symbol Device:R
- added SW2: SW_SPDT, symbol Switch:SW_SPDT
- added U5: MP1475SGJ-P, Package_TO_SOT_SMD:TSOT-23-8, symbol CustomSymbols:MP1475S
Connections:
- net GND: now also BT1.1 (-), BU33SD5WG-TR1.2 (GND), BU33SD5WG-TR2.2 (GND), C1.2, C10.2, C11.2, C12.2, C13.2, C15.2, C18.2, C2.2, C7.2, D1.1 (K), D2.1 (K), D3.2 (A), R13.1, R14.2, U5.1 (PG), U5.4 (GND)
- new net: D1.2 (A), R3.2
- new net: C11.1, C15.1, C16.2, D6.2 (A), L1.1, R12.2
- new net: C14.2, L1.2, U5.3 (SW)
- new net: R9.2, U5.6 (EN/SYNC)
- new net: C13.1, R14.1, U5.7 (VCC)
- new net: C14.1, R10.2
- new net: D3.1 (K), F1.2, SW2.2 (B)
- new net: R10.1, U5.5 (BST)
- new net: R11.1, U5.8 (FB)
- new net: BT1.2 (+), F1.1
- new net: D2.2 (A), R5.2
- new net: C16.1, R11.2, R12.1, R13.2
- new net +3.3V: BU33SD5WG-TR1.5 (VOUT), C18.1, R3.1
- new net +3.3VA: BU33SD5WG-TR2.5 (VOUT), C2.1, R5.1
- new net +5V: BU33SD5WG-TR1.1 (VIN), BU33SD5WG-TR1.3 (~{SHDN}), BU33SD5WG-TR2.1 (VIN), BU33SD5WG-TR2.3 (~{SHDN}), C1.1, C7.1, D6.1 (K)
- new net +BATT: C10.1, C12.1, R9.1, SW2.1 (A), U5.2 (IN)
- no-connect marks 0 -> 1
Other:
- removed sheet Power
- added sheet BT_Module (BT_Module.kicad_sch)
- sheet Accelerometer ports: added ACC_Int1, ACC_Int2, ACC_SCLK, ACC_SDIO, ACC_~{CS}; removed none
- sheet MCU ports: added ACC_Int1, ACC_Int2, ACC_SCLK, ACC_SDIO, ACC_~{CS}, BT_UART_CTS, BT_UART_RTS, BT_UART_RX, BT_UART_TX, BT_~{RST}, MOT1_A, MOT1_B, MOT1_FW, MOT1_Imes, MOT1_REV, MOT2_A, MOT2_B, MOT2_FW, MOT2_Imes, MOT2_REV, ToF_SCL, ToF_SDA, ToF_~{Reset}; removed none
- sheet Motor Sheet ports: added ENC_A, ENC_B, Imes, MOT_FW, MOT_REV; removed none
- sheet Motor Sheet1 ports: added ENC_A, ENC_B, Imes, MOT_FW, MOT_REV; removed none
- sheet ToF ports: added ToF_SCL, ToF_SDA, ToF_~{Reset}; removed none
- note added: "BATTERY CONN"
- note added: "BUCK BATT+ -> 5V"
- note added: "LDO 3V3A"
- note added: "LDO 3V3DC"
- note added: "MCU + connections"
- note added: "POWER"
- note added: "SCHOTTKY OR with USBC VBUS"
- moved on the sheet: H101, H102, H103, H104

Commit message: KSA : PCB G431 :
Parts:
- removed BU33SD5WG-TR2: LM1117DT-3.3, Package_TO_SOT_SMD:SOT-23-5, symbol Regulator_Linear:MCP1802x-xx02xOT
- removed C1, C2: 1u, Capacitor_SMD:C_0603_1608Metric_Pad1.08x0.95mm_HandSolder, symbol Device:C_Small
- removed D2: GR, LED_SMD:LED_0603_1608Metric, symbol Device:LED
- removed R5: 1k, Resistor_SMD:R_0402_1005Metric, symbol Device:R
- F101: renamed from F1; footprint (none) -> Custom:2920L300
- H101, H102, H103, H104: footprint MountingHole:MountingHole_2.5mm_Pad_TopBottom -> MountingHole:MountingHole_3.2mm_M3_DIN965_Pad_TopBottom
- L101: renamed from L1; footprint (none) -> Inductor_SMD:L_APV_ANR5020
- SW101: renamed from SW2; footprint (none) -> Custom:Interrupteur
- renumbered BT1 to BT101, BU33SD5WG-TR1 to BU33SD5WG-TR101, C7 to C101, C12 to C102, C10 to C103, C13 to C104, C18 to C105, C14 to C107, C16 to C108, C15 to C109, C11 to C111, D3 to D101, D1 to D102, D6 to D103, R9 to R101, R14 to R102, R3 to R103, R10 to R104, R11 to R105, R13 to R106, R12 to R107, U5 to U101
Connections:
- net GND: no longer R102.2, U101.1 (PG)
- new net: R102.2, U101.1 (PG)
Other:
- note removed: "LDO 3V3A"

Commit message: On a pas de wiork trtee anyway
Parts:
- removed SW101: SW_SPDT, Custom:Interrupteur, symbol Switch:SW_SPDT
- BT101: footprint Connector_AMASS:AMASS_XT30U-F_1x02_P5.0mm_Vertical -> Connector_JST:JST_XH_B2B-XH-AM_1x02_P2.50mm_Vertical
Connections:
- net +BATT: now also D101.1 (K), F101.2
- no-connect marks 1 -> 0
Changed lines of the file:
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@@
 	)
 	(junction
+		(at 63.5 33.02)
+		(diameter 0)
+		(color 0 0 0 0)
+	)
+	(junction
 		(at 104.14 83.82)
 		(diameter 0)
@@
 	)
 	(junction
-		(at 67.31 30.48)
-		(diameter 0)
-		(color 0 0 0 0)
-	)
-	(junction
 		(at 88.9 95.25)
 		(diameter 0)
@@
 		(color 0 0 0 0)
 	)
-	(no_connect
-		(at 63.5 35.56)
-	)
 	(wire
 		(pts
@@
 	(wire
 		(pts
-			(xy 74.93 29.21) (xy 74.93 30.48)
+			(xy 73.66 31.75) (xy 73.66 33.02)
 		)
 		(stroke
@@
 	(wire
 		(pts
-			(xy 74.93 30.48) (xy 67.31 30.48)
-		)
-		(stroke
-			(width 0)
-			(type default)
-		)
-	)
-	(wire
-		(pts
 			(xy 237.49 81.28) (xy 254 81.28)
 		)
@@
 	(wire
 		(pts
-			(xy 48.26 33.02) (xy 53.34 33.02)
+			(xy 48.26 33.02) (xy 63.5 33.02)
 		)
 		(stroke
@@
 	(wire
 		(pts
-			(xy 88.9 90.17) (xy 88.9 95.25)
+			(xy 63.5 33.02) (xy 73.66 33.02)
 		)
 		(stroke
@@
 	(wire
 		(pts
-			(xy 251.46 153.67) (xy 255.27 153.67)
+			(xy 88.9 90.17) (xy 88.9 95.25)
 		)
 		(stroke
@@
 	(wire
 		(pts
-			(xy 72.39 83.82) (xy 82.55 83.82)
+			(xy 251.46 153.67) (xy 255.27 153.67)
 		)
 		(stroke
@@
 	(wire
 		(pts
-			(xy 201.93 35.56) (xy 212.09 35.56)
+			(xy 72.39 83.82) (xy 82.55 83.82)
 		)
 		(stroke
@@
 	(wire
 		(pts
-			(xy 214.63 33.02) (xy 201.93 33.02)
+			(xy 201.93 35.56) (xy 212.09 35.56)
 		)
 		(stroke
@@
 	(wire
 		(pts
-			(xy 233.68 38.1) (xy 227.33 38.1)
+			(xy 214.63 33.02) (xy 201.93 33.02)
 		)
 		(stroke
@@
 	(wire
 		(pts
-			(xy 67.31 30.48) (xy 63.5 30.48)
+			(xy 233.68 38.1) (xy 227.33 38.1)
 		)
 		(stroke
@@
 	)
 	(symbol
-		(lib_id "Switch:SW_SPDT")
-		(at 58.42 33.02 0)
-		(unit 1)
-		(exclude_from_sim no)
-		(in_bom yes)
-		(on_board yes)
-		(dnp no)
-		(fields_autoplaced yes)
-		(property "Reference" "SW101"
-			(at 58.42 24.13 0)
-			(effects
-				(font
-					(size 1.27 1.27)
-				)
-			)
-		)
-		(property "Value" "SW_SPDT"
-			(at 58.42 26.67 0)
-			(effects
-				(font
-					(size 1.27 1.27)
-				)
-			)
-		)
-		(property "Footprint" "Custom:Interrupteur"
-			(at 58.42 33.02 0)
-			(effects
-				(font
-					(size 1.27 1.27)
-				)
-				(hide yes)
-			)
-		)
-		(property "Datasheet" "~"
-			(at 58.42 40.64 0)
-			(effects
-				(font
-					(size 1.27 1.27)
-				)
-				(hide yes)
-			)
-		)
-		(property "Description" "Switch, single pole double throw"
-			(at 58.42 33.02 0)
-			(effects
-				(font
-					(size 1.27 1.27)
-				)
-				(hide yes)
-			)
-		)
-		(pin "2"
-		)
-		(pin "1"
-		)
-		(pin "3"
-		)
-		(instances
-			(project ""
-				(path "/3d65b2f4-4354-4e18-9b77-809d2b1122a1"
-					(reference "SW101")
-					(unit 1)
-				)
-			)
-		)
-	)
-	(symbol
 		(lib_id "CustomSymbols:MP1475S")
 		(at 60.96 83.82 0)
@@
 			)
 		)
-		(property "Footprint" "Connector_AMASS:AMASS_XT30U-F_1x02_P5.0mm_Vertical"
+		(property "Footprint" "Connector_JST:JST_XH_B2B-XH-AM_1x02_P2.50mm_Vertical"
 			(at 26.67 39.116 90)
 			(effects
@@
 	(symbol
 		(lib_id "power:+BATT")
-		(at 74.93 29.21 0)
+		(at 73.66 31.75 0)
 		(unit 1)
 		(exclude_from_sim no)
@@
 		(fields_autoplaced yes)
 		(property "Reference" "#PWR0111"
-			(at 74.93 33.02 0)
+			(at 73.66 35.56 0)
 			(effects
 				(font
@@
 		)
 		(property "Value" "+BATT"
-			(at 74.93 24.13 0)
+			(at 73.66 26.67 0)
 			(effects
 				(font
@@
 		)
 		(property "Footprint" ""
-			(at 74.93 29.21 0)
+			(at 73.66 31.75 0)
 			(effects
 				(font
@@
 		)
 		(property "Datasheet" ""
-			(at 74.93 29.21 0)
+			(at 73.66 31.75 0)
 			(effects
 				(font
@@
 		)
 		(property "Description" "Power symbol creates a global label with name \"+BATT\""
-			(at 74.93 29.21 0)
+			(at 73.66 31.75 0)
 			(effects
 				(font
@@
 	(symbol
 		(lib_id "power:PWR_FLAG")
-		(at 67.31 30.48 0)
+		(at 63.5 33.02 0)
 		(unit 1)
 		(exclude_from_sim no)
@@
 		(fields_autoplaced yes)
 		(property "Reference" "#FLG0101"
-			(at 67.31 28.575 0)
+			(at 63.5 31.115 0)
 			(effects
 				(font
@@
 		)
 		(property "Value" "PWR_FLAG"
-			(at 67.31 25.4 0)
+			(at 63.5 27.94 0)
 			(effects
 				(font
@@
 		)
 		(property "Footprint" ""
-			(at 67.31 30.48 0)
+			(at 63.5 33.02 0)
 			(effects
 				(font
@@
 		)
 		(property "Datasheet" "~"
-			(at 67.31 30.48 0)
+			(at 63.5 33.02 0)
 			(effects
 				(font
@@
 		)
 		(property "Description" "Special symbol for telling ERC where power comes from"
-			(at 67.31 30.48 0)
+			(at 63.5 33.02 0)
 			(effects
 				(font
@@
 	)
 	(sheet
-		(at 177.8 31.75)
-		(size 24.13 15.24)
+		(at 177.8 30.48)
+		(size 24.13 16.51)
 		(exclude_from_sim no)
 		(in_bom yes)
@@
 		)
 		(property "Sheetname" "Motor Sheet"
-			(at 177.8 31.0384 0)
+			(at 177.8 29.7684 0)
 			(effects
 				(font
@@
 	)
 	(sheet
-		(at 233.68 31.75)
-		(size 24.13 15.24)
+		(at 233.68 30.48)
+		(size 24.13 16.51)
 		(exclude_from_sim no)
 		(in_bom yes)
@@
 		)
 		(property "Sheetname" "Motor Sheet1"
-			(at 233.68 31.0384 0)
+			(at 233.68 29.7684 0)
 			(effects
 				(font

Commit message: check pcb kenny LF
Parts:
- added R1, R2: 100k, Resistor_SMD:R_0402_1005Metric, symbol Device:R_Small
Connections:
- net +3.3V: now also R1.1
- net GND: now also R2.2
- new net MOTOR_VREF: R1.2, R2.1
Other:
- sheet BT_Module ports: added BLE_CONFIG; removed none
- sheet MCU ports: added BLE_CONFIG; removed none
- sheet Motor Sheet ports: added VREF; removed none
- sheet Motor Sheet1 ports: added VREF; removed none
