File: Hardware/Mainboard/projet-chat-ese/ToF.kicad_sch (KiCad schematic)
At the start: 1 part, among them U4 TCA9548APWR

Commit message: [Update] PCB
Parts:
- added J1, J501, J502, J503: Conn_01x04, Connector_JST:JST_EH_B4B-EH-A_1x04_P2.50mm_Vertical, symbol Connector_Generic:Conn_01x04
- added R501, R502, R503, R504, R505, R506, R507, R508, R509, R510, R511: 4k7, symbol Device:R_Small
Connections:
- net GND: now also J1.4 (Pin_4), J501.4 (Pin_4), J502.4 (Pin_4), J503.4 (Pin_4)
- net ToF_SCL: now also R501.2
- net ToF_SDA: now also R502.2
- net ToF_~{Reset}: now also R503.2
- net SD3: now reaches U4.10 (SD3)
- net SD3: now also J503.3 (Pin_3), R510.2
- net SC3: now reaches U4.11 (SC3)
- net SC3: now also J503.2 (Pin_2), R511.2
- net SD0: now reaches U4.4 (SD0)
- net SD0: now also J1.3 (Pin_3), R504.2
- net SC0: now reaches U4.5 (SC0)
- net SC0: now also J1.2 (Pin_2), R505.2
- net SD1: now reaches U4.6 (SD1)
- net SD1: now also J501.3 (Pin_3), R506.2
- net SC1: now reaches U4.7 (SC1)
- net SC1: now also J501.2 (Pin_2), R507.2
- net SD2: now reaches U4.8 (SD2)
- net SD2: now also J502.3 (Pin_3), R508.2
- net SC2: now reaches U4.9 (SC2)
- net SC2: now also J502.2 (Pin_2), R509.2
- new net +3.3V: J1.1 (Pin_1), J501.1 (Pin_1), J502.1 (Pin_1), J503.1 (Pin_1), R501.1, R502.1, R503.1, R504.1, R505.1, R506.1, R507.1, R508.1, R509.1, R510.1, R511.1
- no-connect marks 0 -> 8
Other:
- note added: "Connecteurs ToF"

Commit message: KSA : PCB G431 :
Parts:
- R501: renamed from R502; footprint (none) -> Resistor_SMD:R_0402_1005Metric
- R502: renamed from R503; footprint (none) -> Resistor_SMD:R_0402_1005Metric
- R503: renamed from R501; footprint (none) -> Resistor_SMD:R_0402_1005Metric
- R504: renamed from R508; footprint (none) -> Resistor_SMD:R_0402_1005Metric
- R505: renamed from R504; footprint (none) -> Resistor_SMD:R_0402_1005Metric
- R506: renamed from R509; footprint (none) -> Resistor_SMD:R_0402_1005Metric
- R507: renamed from R505; footprint (none) -> Resistor_SMD:R_0402_1005Metric
- R508: renamed from R510; footprint (none) -> Resistor_SMD:R_0402_1005Metric
- R509: renamed from R506; footprint (none) -> Resistor_SMD:R_0402_1005Metric
- R510: renamed from R511; footprint (none) -> Resistor_SMD:R_0402_1005Metric
- R511: renamed from R507; footprint (none) -> Resistor_SMD:R_0402_1005Metric
- renumbered J502 to J501, J1 to J502, J501 to J504, U4 to U501

Commit message: On a pas de wiork trtee anyway
Parts:
- J501, J502, J503, J504: footprint Connector_JST:JST_EH_B4B-EH-A_1x04_P2.50mm_Vertical -> Connector_JST:JST_PH_B4B-PH-K_1x04_P2.00mm_Vertical
- U501: footprint Package_SO:TSSOP-24_4.4x7.8mm_P0.65mm -> Package_DFN_QFN:VQFN-24-1EP_4x4mm_P0.5mm_EP2.45x2.45mm
Changed lines of the file:
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@@
 			)
 		)
-		(property "Footprint" "Package_SO:TSSOP-24_4.4x7.8mm_P0.65mm"
+		(property "Footprint" "Package_DFN_QFN:VQFN-24-1EP_4x4mm_P0.5mm_EP2.45x2.45mm"
 			(at 57.15 99.06 0)
 			(effects
@@
 			)
 		)
-		(property "Footprint" "Connector_JST:JST_EH_B4B-EH-A_1x04_P2.50mm_Vertical"
+		(property "Footprint" "Connector_JST:JST_PH_B4B-PH-K_1x04_P2.00mm_Vertical"
 			(at 185.42 62.23 0)
 			(effects
@@
 			)
 		)
-		(property "Footprint" "Connector_JST:JST_EH_B4B-EH-A_1x04_P2.50mm_Vertical"
+		(property "Footprint" "Connector_JST:JST_PH_B4B-PH-K_1x04_P2.00mm_Vertical"
 			(at 137.16 87.63 0)
 			(effects
@@
 			)
 		)
-		(property "Footprint" "Connector_JST:JST_EH_B4B-EH-A_1x04_P2.50mm_Vertical"
+		(property "Footprint" "Connector_JST:JST_PH_B4B-PH-K_1x04_P2.00mm_Vertical"
 			(at 138.43 62.23 0)
 			(effects
@@
 			)
 		)
-		(property "Footprint" "Connector_JST:JST_EH_B4B-EH-A_1x04_P2.50mm_Vertical"
+		(property "Footprint" "Connector_JST:JST_PH_B4B-PH-K_1x04_P2.00mm_Vertical"
 			(at 184.15 87.63 0)
 			(effects

Commit message: Last PCB edits G431
Connections:
- net GND: now also U501.25 (PAD)
Changed lines of the file:
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@@
 		(pin "19"
+		)
+		(pin "25"
 		)
 		(instances
