File: Hardware/Mainboard/projet-chat-ese/motor.kicad_sch (KiCad schematic)
At the start: 6 parts

Commit message: [Update] PCB
Parts:
- added U7: GO 10-SME/SP3, Package_SO:SOIC-8-1EP_3.9x4.9mm_P1.27mm_EP2.41x3.3mm, symbol Custom:GO_10-SME
- J201: renamed from J; footprint (none) -> Connector_JST:JST_EH_B6B-EH-A_1x06_P2.50mm_Vertical
- R201: renamed from R; footprint (none) -> Resistor_SMD:R_0402_1005Metric
- R8: footprint (none) -> Resistor_SMD:R_0402_1005Metric
- U201: renamed from U; footprint SOIC8_ZXBM5210-SP-13_DIO -> Package_SO:SOIC-8-1EP_3.9x4.9mm_P1.27mm_EP2.29x3mm
- renumbered C to C201
Connections:
- net +3.3V: now also U7.8 (UC)
- net GND: now also U7.5 (GND)
- net MOT+: now also U7.1 (IP+), U7.2 (IP+); no longer J201.1 (Pin_1)
- new net Imes: U7.7 (UOUT)
- new net MOT+_OUT: J201.1 (Pin_1), U7.3 (IP-), U7.4 (IP-)
- no-connect marks 0 -> 1
Other:
- note added: "Hall Sensor"

Commit message: KSA : PCB G431 :
Parts:
- added C203: 4.7n, Capacitor_SMD:C_0402_1005Metric, symbol Device:C_Small
- added C604: 47n, Capacitor_SMD:C_0402_1005Metric, symbol Device:C_Small
- renumbered C9 to C202, R8 to R201, R201 to R202, U7 to U202
Connections:
- net +3.3V: now also C604.1
- net GND: now also C203.2, C604.2
- net Imes: now also C203.1
- net +5V renamed +BATT

Commit message: On a pas de wiork trtee anyway
Parts:
- removed C604: 47n, Capacitor_SMD:C_0402_1005Metric, symbol Device:C_Small
- removed U202: GO 10-SME/SP3, Package_SO:SOIC-8-1EP_3.9x4.9mm_P1.27mm_EP2.41x3.3mm, symbol Custom:GO_10-SME
- added R203: 10m, Resistor_SMD:R_0805_2012Metric, symbol Device:R_Small
- added U202: NCS199A3RSQT2G, Custom:SC70-6, symbol CustomSymbols:NCS199A3RSQT2G
- C203: value 4.7n -> 100n
- J201: footprint Connector_JST:JST_EH_B6B-EH-A_1x06_P2.50mm_Vertical -> Connector_JST:JST_PH_B6B-PH-K_1x06_P2.00mm_Vertical
Connections:
- net +3.3V: now also C203.2, U202.3 (VS)
- net GND: now also C203.1, U202.1 (Vref), U202.2 (GND); no longer C203.2
- net Imes: now also U202.6 (OUT); no longer C203.1
- net MOT+: now also R203.1, U202.5 (IN-)
- net MOT+_OUT: now also R203.2, U202.4 (IN+)
- no-connect marks 1 -> 0
Other:
- note added: "Shunt Current Sensor"
- note removed: "Hall Sensor"

Commit message: Finishing PCB
Connections:
- net GND: now also U201.9 (GND)
Changed lines of the file:
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@@
 		(pin "5"
+		)
+		(pin "9"
 		)
 		(instances

Commit message: check pcb kenny LF
Parts:
- removed R201, R202: R_Small, Resistor_SMD:R_0402_1005Metric, symbol Device:R_Small
Connections:
- net +BATT: now also U201.6 (VREF)
- net GND: no longer U202.1 (Vref)
- new net VREF: U202.1 (Vref)
Other:
- note removed: "DEFINIR LE PONT DIVISEUR"
- moved on the sheet: C201, C202

Commit message: Kenny's Last work
Parts:
- renumbered J201 to J601
Connections:
- net +3.3V: now also J601.2 (Pin_2); no longer J601.5 (Pin_5)
- net ENC_A: now also J601.4 (Pin_4); no longer J601.3 (Pin_3)
- net ENC_B: now also J601.3 (Pin_3); no longer J601.4 (Pin_4)
- net GND: now also J601.5 (Pin_5); no longer J601.2 (Pin_2)
- net MOT+_OUT: now also J601.6 (Pin_6); no longer J601.1 (Pin_1)
- net MOT-: now also J601.1 (Pin_1); no longer J601.6 (Pin_6)
Changed lines of the file:
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@@
 	(symbol
 		(lib_id "Connector:Conn_01x06_Socket")
-		(at 210.82 43.18 0)
+		(at 210.82 45.72 0)
+		(mirror x)
 		(unit 1)
 		(exclude_from_sim no)
@@
 		(on_board yes)
 		(dnp no)
-		(fields_autoplaced yes)
-		(property "Reference" "J201"
-			(at 212.09 43.1799 0)
+		(property "Reference" "J601"
+			(at 212.09 45.7201 0)
 			(effects
 				(font
@@
 		)
 		(property "Value" "Conn_01x06_Socket"
-			(at 212.09 45.7199 0)
+			(at 212.09 43.1801 0)
 			(effects
 				(font
@@
 		)
 		(property "Footprint" "Connector_JST:JST_PH_B6B-PH-K_1x06_P2.00mm_Vertical"
-			(at 210.82 43.18 0)
+			(at 210.82 45.72 0)
 			(effects
 				(font
@@
 		)
 		(property "Datasheet" "~"
-			(at 210.82 43.18 0)
+			(at 210.82 45.72 0)
 			(effects
 				(font
@@
 		)
 		(property "Description" "Generic connector, single row, 01x06, script generated"
-			(at 210.82 43.18 0)
+			(at 210.82 45.72 0)
 			(effects
 				(font
@@
 			(project "projet-chat-ese"
 				(path "/3d65b2f4-4354-4e18-9b77-809d2b1122a1/afd2bf17-892c-4de5-9c32-bb69ff013475"
-					(reference "J201")
+					(reference "J601")
 					(unit 1)
 				)
 				(path "/3d65b2f4-4354-4e18-9b77-809d2b1122a1/dbb36908-5e11-4a5e-b84d-3e3df0bcdb8e"
-					(reference "J601")
+					(reference "J602")
 					(unit 1)
 				)
