File: Hardware/Bluetooth/STM32WB55/untitled.kicad_sch (KiCad schematic)
At the start: 49 parts, among them J1 Conn_ST_STDC14, J11 Conn_01x06, J14 Conn_01x06, J2 Conn_01x04, SW2 SW_SPST, U1 STM32WB55CGUx, X1 32kHz758, Y2 Crystal_GND24_Small

Commit message: schematic update
Other:
- note added: "Half of the max speed"
- note added: "JTAG Connector"
- note removed: "PWM motor to GND to be at the minimum speed"
Changed lines of the file:
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@@
 	(paper "A4")
 	(rectangle
-		(start 11.938 11.938)
-		(end 57.912 58.42)
+		(start 21.59 138.43)
+		(end 66.04 190.5)
 		(stroke
-			(width 0)
-			(type default)
+			(width 1)
+			(type solid)
 		)
 		(fill
@@
 	(text "ST_LINK\n"
 		(exclude_from_sim no)
-		(at 19.812 16.256 0)
+		(at 33.02 147.32 0)
 		(effects
 			(font
@@
 		)
 	)
+	(text "JTAG Connector\n"
+		(exclude_from_sim no)
+		(at 43.18 135.89 0)
+		(effects
+			(font
+				(size 2 2)
+				(thickness 0.4)
+				(bold yes)
+			)
+		)
+	)
 	(text "Lidar"
 		(exclude_from_sim no)
@@
 		)
 	)
-	(text "PWM motor to GND to\n be at the minimum speed"
+	(text "Half of the max speed\n"
 		(exclude_from_sim no)
-		(at 215.9 116.84 0)
+		(at 220.98 128.27 0)
 		(effects
 			(font
@@
 	)
 	(junction
-		(at 35.56 52.07)
+		(at 41.91 182.88)
 		(diameter 0)
 		(color 0 0 0 0)
@@
 	)
 	(no_connect
-		(at 48.26 34.29)
+		(at 54.61 165.1)
 	)
 	(no_connect
-		(at 48.26 46.99)
+		(at 54.61 177.8)
 	)
 	(no_connect
@@
 	)
 	(no_connect
-		(at 48.26 39.37)
+		(at 54.61 170.18)
 	)
 	(no_connect
@@
 	)
 	(no_connect
-		(at 48.26 44.45)
+		(at 54.61 175.26)
 	)
 	(no_connect
@@
 	(wire
 		(pts
-			(xy 54.61 26.67) (xy 48.26 26.67)
+			(xy 60.96 157.48) (xy 54.61 157.48)
 		)
 		(stroke
@@
 	(wire
 		(pts
-			(xy 48.26 21.59) (xy 54.102 21.59)
+			(xy 54.61 152.4) (xy 60.452 152.4)
 		)
 		(stroke
@@
 	(wire
 		(pts
-			(xy 54.61 31.75) (xy 48.26 31.75)
+			(xy 60.96 162.56) (xy 54.61 162.56)
 		)
 		(stroke
@@
 	(wire
 		(pts
-			(xy 33.02 52.07) (xy 35.56 52.07)
+			(xy 39.37 182.88) (xy 41.91 182.88)
 		)
 		(stroke
@@
 	(wire
 		(pts
-			(xy 54.61 29.21) (xy 48.26 29.21)
+			(xy 60.96 160.02) (xy 54.61 160.02)
 		)
 		(stroke
@@
 	)
 	(label "SWO"
-		(at 54.61 31.75 180)
+		(at 60.96 162.56 180)
 		(effects
 			(font
@@
 	)
 	(label "SWCLK"
-		(at 54.61 26.67 180)
+		(at 60.96 157.48 180)
 		(effects
 			(font
@@
 	)
 	(label "NRST"
-		(at 54.102 21.59 180)
+		(at 60.452 152.4 180)
 		(effects
 			(font
@@
 	)
 	(label "SWDIO"
-		(at 54.61 29.21 180)
+		(at 60.96 160.02 180)
 		(effects
 			(font
@@
 	(symbol
 		(lib_id "power:GND")
-		(at 35.56 52.07 0)
+		(at 41.91 182.88 0)
 		(unit 1)
 		(exclude_from_sim no)
@@
 		(fields_autoplaced yes)
 		(property "Reference" "#PWR090"
-			(at 35.56 58.42 0)
+			(at 41.91 189.23 0)
 			(effects
 				(font
@@
 		)
 		(property "Value" "GND"
-			(at 35.56 57.15 0)
+			(at 41.91 187.96 0)
 			(effects
 				(font
@@
 		)
 		(property "Footprint" ""
-			(at 35.56 52.07 0)
+			(at 41.91 182.88 0)
 			(effects
 				(font
@@
 		)
 		(property "Datasheet" ""
-			(at 35.56 52.07 0)
+			(at 41.91 182.88 0)
 			(effects
 				(font
@@
 		)
 		(property "Description" "Power symbol creates a global label with name \"GND\" , ground"
-			(at 35.56 52.07 0)
+			(at 41.91 182.88 0)
 			(effects
 				(font
@@
 	(symbol
 		(lib_id "power:+3.3V")
-		(at 35.56 16.51 0)
+		(at 41.91 147.32 0)
 		(unit 1)
 		(exclude_from_sim no)
@@
 		(dnp no)
 		(property "Reference" "#PWR089"
-			(at 35.56 20.32 0)
+			(at 41.91 151.13 0)
 			(effects
 				(font
@@
 		)
 		(property "Value" "+3.3V"
-			(at 38.862 12.954 0)
+			(at 45.212 143.764 0)
 			(effects
 				(font
@@
 		)
 		(property "Footprint" ""
-			(at 35.56 16.51 0)
+			(at 41.91 147.32 0)
 			(effects
 				(font
@@
 		)
 		(property "Datasheet" ""
-			(at 35.56 16.51 0)
+			(at 41.91 147.32 0)
 			(effects
 				(font
@@
 		)
 		(property "Description" "Power symbol creates a global label with name \"+3.3V\""
-			(at 35.56 16.51 0)
+			(at 41.91 147.32 0)
 			(effects
 				(font
@@
 	(symbol
 		(lib_id "Connector:Conn_ST_STDC14")
-		(at 35.56 34.29 0)
+		(at 41.91 165.1 0)
 		(unit 1)
 		(exclude_from_sim no)
@@
 		(fields_autoplaced yes)
 		(property "Reference" "J1"
-			(at 24.892 33.0199 0)
+			(at 31.242 163.8299 0)
 			(effects
 				(font
@@
 				)
 				(justify right)
+				(hide yes)
 			)
 		)
 		(property "Value" "Conn_ST_STDC14"
-			(at 24.892 35.5599 0)
+			(at 31.242 166.3699 0)
 			(effects
 				(font
@@
 				)
 				(justify right)
+				(hide yes)
 			)
 		)
 		(property "Footprint" "Connector_PinHeader_1.27mm:PinHeader_2x07_P1.27mm_Vertical_SMD"
-			(at 35.56 34.29 0)
+			(at 41.91 165.1 0)
 			(effects
 				(font
@@
 		)
 		(property "Datasheet" "https://www.st.com/content/ccc/resource/technical/document/user_manual/group1/99/49/91/b6/b2/3a/46/e5/DM00526767/files/DM00526767.pdf/jcr:content/translations/en.DM00526767.pdf"
-			(at 26.67 66.04 90)
+			(at 33.02 196.85 90)
 			(effects
 				(font
@@
 		)
 		(property "Description" "ST Debug Connector, standard ARM Cortex-M SWD and JTAG interface plus UART"
-			(at 35.56 34.29 0)
+			(at 41.91 165.1 0)
 			(effects
 				(font
@@
 					(size 1.27 1.27)
 				)
+				(hide yes)
 			)
 		)
