File: Hardware/Bluetooth/STM32WB55/I2C.kicad_sch (KiCad schematic)
At the start: 20 parts, among them J3 Conn_01x04, J4 Conn_01x04, J5 Conn_01x04, J6 Conn_01x04, J7 Conn_01x04, J8 Conn_01x04, U3 ADXL343, U4 TCA9548AMRGER

Commit message: schematic update
Connections:
- net I2C_SCL: now also U4.19 (SCL); no longer U4.20 (SDA)
- net I2C_SDA: now also U4.20 (SDA); no longer U4.19 (SCL)
Other:
- note added: "3 Axes"
- note added: "Connecteurs"
- note added: "Multiplexer"
- note removed: "6-AXIS"
- moved on the sheet: R1, R2, R20, R3, R30, R5, U3, U4

Commit message: clean
Changed lines of the file:
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@@
-	(wire
-		(pts
-			(xy 38.1 137.16) (xy 50.546 137.16)
-		)
-		(stroke
-			(width 0)
-			(type default)
-		)
-	)
 	(wire
 		(pts
@@
 	(wire
 		(pts
-			(xy 50.546 140.97) (xy 50.8 140.97)
-		)
-		(stroke
-			(width 0)
-			(type default)
-		)
-	)
-	(wire
-		(pts
 			(xy 207.01 87.63) (xy 201.93 87.63)
 		)
@@
 		(pts
 			(xy 54.61 127) (xy 58.42 127)
-		)
-		(stroke
-			(width 0)
-			(type default)
-		)
-	)
-	(wire
-		(pts
-			(xy 50.546 137.16) (xy 50.546 140.97)
 		)
 		(stroke
@@
 	(symbol
 		(lib_id "power:GND")
-		(at 38.1 137.16 0)
+		(at 50.8 140.97 270)
 		(unit 1)
 		(exclude_from_sim no)
@@
 		(dnp no)
 		(property "Reference" "#PWR057"
-			(at 38.1 143.51 0)
+			(at 44.45 140.97 0)
 			(effects
 				(font
@@
 		)
 		(property "Value" "GND"
-			(at 34.29 137.922 0)
+			(at 50.038 137.16 0)
 			(effects
 				(font
@@
 		)
 		(property "Footprint" ""
-			(at 38.1 137.16 0)
+			(at 50.8 140.97 0)
 			(effects
 				(font
@@
 		)
 		(property "Datasheet" ""
-			(at 38.1 137.16 0)
+			(at 50.8 140.97 0)
 			(effects
 				(font
@@
 		)
 		(property "Description" "Power symbol creates a global label with name \"GND\" , ground"
-			(at 38.1 137.16 0)
-			(effects
-				(font
+			(at 50.8 140.97 0)
+			(effects
+				(font
