File: Hardware/Bluetooth/STM32WB55/Main_Board.kicad_pcb (KiCad board)
At the start: 4 copper layers, 64 x 41.8 mm, 110 parts, among them IC2 MP1475SGJ-P, IC3 ZXBM5210-SP-13, IC4 ZXBM5210-SP-13, J1 Conn_ST_STDC14, J11 Conn_01x06, J14 Conn_01x06, J2 Conn_01x04, J3 Conn_01x04, J4 Conn_01x04, J5 Conn_01x04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

Commit message: clean
Connections:
- net /OUT_BUTTON renamed /Converters/OUT_BUTTON
- net /V_bat renamed /Converters/V_bat
- U4 pad 19: /I2C_SDA -> /I2C_SCL
- U4 pad 20: /I2C_SCL -> /I2C_SDA
Routing:
- net /I2C_SCL: track 40.6 -> 41.7 mm
Changed lines of the file:
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@@
 			(drillshape 0)
 			(scaleselection 1)
-			(outputdirectory "../../../../PROJET_ESE_ROBOT_CHAT/Hardware/Bluetooth/Board_STM32WB55/")
+			(outputdirectory "../Gerber/")
 		)
 	)
@@
 	(net 54 "/I2C_SCL")
 	(net 55 "/I2C_SDA")
-	(net 56 "/V_bat")
-	(net 57 "/OUT_BUTTON")
+	(net 56 "/Converters/V_bat")
+	(net 57 "/Converters/OUT_BUTTON")
 	(net 58 "/STM32/ENCODEUR_A_M1")
 	(net 59 "/STM32/ENCODEUR_B_M1")
@@
 			(layers "F.Cu" "F.Mask" "F.Paste")
 			(roundrect_rratio 0.25)
-			(net 55 "/I2C_SDA")
+			(net 54 "/I2C_SCL")
 			(pinfunction "SCL")
 			(pintype "input")
@@
 			(layers "F.Cu" "F.Mask" "F.Paste")
 			(roundrect_rratio 0.25)
-			(net 54 "/I2C_SCL")
+			(net 55 "/I2C_SDA")
 			(pinfunction "SDA")
 			(pintype "bidirectional")
@@
 		)
 		(property ki_fp_filters "Connector*:*_1x??_*")
-		(sheetname "/")
-		(sheetfile "Main_Board.kicad_sch")
+		(sheetname "/Converters/")
+		(sheetfile "converters.kicad_sch")
 		(attr through_hole)
 		(fp_line
@@
 			(remove_unused_layers no)
 			(roundrect_rratio 0.147059)
-			(net 56 "/V_bat")
+			(net 56 "/Converters/V_bat")
 			(pinfunction "Pin_1")
 			(pintype "passive")
@@
 		)
 		(property ki_fp_filters "*WS-TOTV*472121010111*")
-		(sheetname "/")
-		(sheetfile "Main_Board.kicad_sch")
+		(sheetname "/Converters/")
+		(sheetfile "converters.kicad_sch")
 		(attr through_hole)
 		(fp_line
@@
 			(layers "*.Cu" "*.Mask")
 			(remove_unused_layers no)
-			(net 57 "/OUT_BUTTON")
+			(net 57 "/Converters/OUT_BUTTON")
 			(pinfunction "1")
 			(pintype "passive")
@@
 			(layers "*.Cu" "*.Mask")
 			(remove_unused_layers no)
-			(net 56 "/V_bat")
+			(net 56 "/Converters/V_bat")
 			(pinfunction "2")
 			(pintype "passive")
@@
 		)
 		(property ki_fp_filters "C_*")
-		(sheetname "/")
-		(sheetfile "Main_Board.kicad_sch")
+		(sheetname "/Converters/")
+		(sheetfile "converters.kicad_sch")
 		(attr smd)
 		(fp_line
@@
 		)
 		(property ki_fp_filters "R_*")
-		(sheetname "/")
-		(sheetfile "Main_Board.kicad_sch")
+		(sheetname "/Converters/")
+		(sheetfile "converters.kicad_sch")
 		(attr smd)
 		(fp_line
@@
 		)
 		(property ki_fp_filters "R_*")
-		(sheetname "/")
-		(sheetfile "Main_Board.kicad_sch")
+		(sheetname "/Converters/")
+		(sheetfile "converters.kicad_sch")
 		(attr smd)
 		(fp_line
@@
 		)
 		(property ki_fp_filters "TSSOP*4.4x3mm*P0.65mm*")
-		(sheetname "/")
-		(sheetfile "Main_Board.kicad_sch")
+		(sheetname "/Converters/")
+		(sheetfile "converters.kicad_sch")
 		(attr smd)
 		(fp_line
@@
 			(layers "B.Cu" "B.Mask" "B.Paste")
 			(roundrect_rratio 0.25)
-			(net 57 "/OUT_BUTTON")
+			(net 57 "/Converters/OUT_BUTTON")
 			(pinfunction "+")
 			(pintype "input")
@@
 		)
 		(property ki_fp_filters "R_*")
-		(sheetname "/")
-		(sheetfile "Main_Board.kicad_sch")
+		(sheetname "/Converters/")
+		(sheetfile "converters.kicad_sch")
 		(attr smd)
 		(fp_line
@@
 			(size 2.9 3.3)
 			(layers "B.Cu" "B.Mask" "B.Paste")
-			(net 57 "/OUT_BUTTON")
+			(net 57 "/Converters/OUT_BUTTON")
 			(pintype "passive")
 		)
@@
 	)
 	(segment
-		(start 55.580015 154.432)
-		(end 56.178015 153.834)
-		(width 0.18)
-		(layer "F.Cu")
-		(net 54)
-	)
-	(segment
 		(start 64.18 150.07696)
 		(end 63.979 150.27796)
@@
 	)
 	(segment
-		(start 56.178015 153.834)
-		(end 57.584 153.834)
-		(width 0.18)
-		(layer "F.Cu")
-		(net 54)
-	)
-	(segment
 		(start 69.5 147.050002)
 		(end 69.5 147.242104)
@@
 	)
 	(segment
-		(start 53.7972 154.432)
-		(end 55.580015 154.432)
-		(width 0.18)
-		(layer "F.Cu")
-		(net 54)
-	)
-	(segment
 		(start 69.2885 147.7385)
 		(end 69.381105 147.831105)
@@
 	)
 	(segment
-		(start 52.75 152)
-		(end 52.75 153.3848)
-		(width 0.18)
-		(layer "F.Cu")
-		(net 54)
-	)
-	(segment
 		(start 69.2885 147.453604)
 		(end 69.2885 147.7385)
@@
 	)
 	(segment
-		(start 52.75 153.3848)
-		(end 53.7972 154.432)
-		(width 0.18)
+		(start 55.159958 156.376)
+		(end 52.25 153.466042)
+		(width 0.2)
 		(layer "F.Cu")
 		(net 54)
@@
 	)
 	(segment
-		(start 76.425 144.6875)
-		(end 76.425 145.325)
-		(width 0.19)
+		(start 58.75 155.2)
+		(end 57.574 156.376)
+		(width 0.2)
 		(layer "F.Cu")
 		(net 54)
 	)
 	(segment
-		(start 57.584 153.834)
-		(end 58.75 155)
-		(width 0.18)
+		(start 76.425 144.6875)
+		(end 76.425 145.325)
+		(width 0.19)
 		(layer "F.Cu")
 		(net 54)
@@
 	)
 	(segment
+		(start 52.25 153.466042)
+		(end 52.25 152)
+		(width 0.2)
+		(layer "F.Cu")
+		(net 54)
+	)
+	(segment
 		(start 63.979 150.27796)
 		(end 63.979 152.251)
@@
 	)
 	(segment
+		(start 57.574 156.376)
+		(end 55.159958 156.376)
+		(width 0.2)
+		(layer "F.Cu")
+		(net 54)
+	)
+	(segment
 		(start 64.521 148.279)
 		(end 64.18 148.62)
@@
 	)
 	(segment
-		(start 52.25 152)
-		(end 52.25 153.4944)
-		(width 0.18)
+		(start 54.551058 155.2)
+		(end 56.75 155.2)
+		(width 0.2)
 		(layer "F.Cu")
 		(net 55)
@@
 	)
 	(segment
+		(start 52.75 153.398942)
+		(end 54.551058 155.2)
+		(width 0.2)
+		(layer "F.Cu")
+		(net 55)
+	)
+	(segment
 		(start 71.2885 148.253604)
 		(end 71.2885 148.931396)
@@
 	)
 	(segment
-		(start 53.7556 155)
-		(end 56.75 155)
-		(width 0.18)
+		(start 52.75 152)
+		(end 52.75 153.398942)
+		(width 0.2)
 		(layer "F.Cu")
 		(net 55)
@@
 	)
 	(segment
-		(start 52.25 153.4944)
-		(end 53.7556 155)
-		(width 0.18)
-		(layer "F.Cu")
-		(net 55)
-	)
-	(segment
 		(start 76.925 145.975)
 		(end 76.7 146.2)
@@
 	)
 	(segment
+		(start 60.85 146)
+		(end 61.6 146)
+		(width 0.2)
+		(layer "B.Cu")
+		(net 62)
+	)
+	(segment
 		(start 76.913128 144.006)
 		(end 74.607128 141.7)
@@
 	(segment
 		(start 61.6 146)
-		(end 62.275 145.325)
-		(width 0.19)
+		(end 61.994986 145.605014)
+		(width 0.2)
 		(layer "B.Cu")
 		(net 62)
@@
 	)
 	(segment
-		(start 60.85 146)
-		(end 61.6 146)
-		(width 0.19)
-		(layer "B.Cu")
-		(net 62)
-	)
-	(segment
 		(start 54.76 152.01)
 		(end 54.75 152)
@@
 	(zone
 		(net 57)
-		(net_name "/OUT_BUTTON")
+		(net_name "/Converters/OUT_BUTTON")
 		(layer "F.Cu")
 		(hatch edge 0.5)
@@
 	(zone
 		(net 57)
-		(net_name "/OUT_BUTTON")
+		(net_name "/Converters/OUT_BUTTON")
 		(layer "B.Cu")
 		(hatch edge 0.5)
